File: manufacturing/USBC-PowerSwitcher/Digital.kicad_sch (KiCad schematic)
At the start: 16 parts, among them U1 STM32F412RGT6

Commit message: First Rough placement
Parts:
- C1, C15, C2, C8: footprint (none) -> Capacitor_SMD:C_0805_2012Metric; LCSC # (none) -> C1779
- C11, C3, C4, C5, C6, C7: footprint (none) -> Capacitor_SMD:C_0402_1005Metric; LCSC # (none) -> C307331
- FB1: footprint (none) -> Inductor_SMD:L_0805_2012Metric; LCSC # (none) -> C1015
- R4, R5, R6: footprint Resistor_SMD:R_0805_2012Metric_Pad1.20x1.40mm_HandSolder -> Resistor_SMD:R_0402_1005Metric; LCSC # (none) -> C25879
- U1: LCSC # (none) -> C94351
Connections:
- net +3V3: now also U1.1 (VBAT)
- net ADC1_IN0: no longer names the net of U1.14 (PA0)
- net ADC1_IN1: no longer names the net of U1.15 (PA1)
- net PD_GPIO: no longer names the net of U1.38 (PC7)
- no-connect marks 0 -> 28
Other:
- note added: "16MHz"
- note added: "SWD"
- moved on the sheet: C11, C4, C5, C6, C7, C8
